File: PCBs/TarjetasDeDesarrollo/PectenAlpha/PectenAlphaSMD/PectenAlphaSMD.kicad_pcb (KiCad board)
At the start: 2 copper layers, 50 x 50 mm, 27 parts, among them J1 ICSP, J3 USB_A, J4 PORT, J5 EXPANSION, SW1 SW_Push, SW2 SW_DIP_x04, U1 PIC_8-14-18-20, U2 D148K, U3 CH340N, U4 AMS1117-3.3

Commit message: Tarjeta Pecten
Parts:
- removed J3: USB_A, Connector_USB:USB_A_CNCTech_1001-011-01101_Horizontal
- removed J4: PORT, Connector_PinHeader_2.54mm:PinHeader_2x12_P2.54mm_Vertical
- removed J5: EXPANSION, Connector_PinHeader_2.54mm:PinHeader_2x08_P2.54mm_Vertical
- removed R16: R_US, Resistor_SMD:R_0805_2012Metric_Pad1.20x1.40mm_HandSolder
- removed SW2: SW_DIP_x04, Button_Switch_THT:SW_DIP_SPSTx04_Slide_6.7x11.72mm_W7.62mm_P2.54mm_LowProfile
- added BZ1: Buzzer, Buzzer_Beeper:Buzzer_12x9.5RM7.6, F.Cu at (110.8, 50.0)
- added C2: 10uF, Capacitor_SMD:CP_Elec_5x3, F.Cu at (118.6, 46.7)
- added C3: 100uF, Capacitor_SMD:CP_Elec_5x3, F.Cu at (114.2, 42.2)
- added J2: PectenExpansionPort, PIC_Pin_Compatible:PXP, F.Cu at (150.0, 80.0)
- added Q2: PN2222A, Package_TO_SOT_THT:TO-92_Inline, F.Cu at (115.0, 54.0)
- added R14: R_US, Resistor_SMD:R_0805_2012Metric_Pad1.20x1.40mm_HandSolder, F.Cu at (115.8, 57.8)
- added SW3: SW_DIP_x01, Button_Switch_THT:SW_DIP_SPSTx01_Slide_6.7x4.1mm_W7.62mm_P2.54mm_LowProfile, F.Cu at (102.8, 64.1)
- added SW4: SW_DIP_x01, Button_Switch_THT:SW_DIP_SPSTx01_Slide_6.7x4.1mm_W7.62mm_P2.54mm_LowProfile, F.Cu at (102.8, 73.9)
- added U5: 74HC595, Package_SO:SOP-16_4.4x10.4mm_P1.27mm, F.Cu at (138.1, 55.1)
- R1, R10, R11, R12, R13, R2, R3, R4, R5, R6, R7, R8, R9: moved to B.Cu
- R15: moved to F.Cu
- U3: value CH340N -> 74HC595; footprint Package_SO:JEITA_SOIC-8_3.9x4.9mm_P1.27mm -> Package_SO:SOP-16_4.4x10.4mm_P1.27mm; moved to F.Cu
- moved R1 68.5 mm to (117.0, 32.0), turned to 180 degrees
- moved R8 51.1 mm to (109.4, 66.8), turned to 180 degrees
- moved R10 51.1 mm to (127.0, 60.5), turned to 90 degrees
- moved R7 50.4 mm to (109.4, 64.8), turned to 180 degrees
- moved R13 47.7 mm to (119.8, 66.0), turned to -90 degrees
- moved R12 47.7 mm to (123.0, 60.5), turned to 90 degrees
- moved R3 45.9 mm to (114.7, 64.8), turned to 180 degrees
- moved R5 45.7 mm to (109.4, 75.5), turned to 180 degrees
- moved R11 44.1 mm to (125.0, 60.5), turned to 90 degrees
- moved R9 43.5 mm to (114.4, 75.5), turned to 180 degrees
- moved R6 43.4 mm to (109.4, 73.5), turned to 180 degrees
- moved J1 42.6 mm to (103.6, 42.4), turned to 135 degrees
- moved R2 42.0 mm to (114.7, 66.8), turned to 180 degrees
- moved R4 41.6 mm to (114.4, 73.5), turned to 180 degrees
- moved D1 39.9 mm to (116.2, 32.7), turned to -45 degrees
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Connections:
- D10 pad 3: /LED RGB -> /pxp
- J1 pad 5: +5V -> VCC
- J1 pad 6: Net-(J1-Pin_6) -> /RA4/RA4
- R10 pad 1: /RA0/RA0 -> /GPB2
- R11 pad 1: /RA1/RA7 -> /GPB1
- R12 pad 1: /RA2/RA6 -> /GPB0
- R15 pad 1: Net-(JP1-C) -> /pxpcs
- R15 pad 2: Net-(U3-TXD) -> +5V
- R2 pad 1: unconnected-(R2-Pad1) -> /GPA0
- R3 pad 1: unconnected-(R3-Pad1) -> /GPA1
- R4 pad 1: unconnected-(R4-Pad1) -> /GPA2
- R5 pad 1: unconnected-(R5-Pad1) -> /GPA3
- R6 pad 1: unconnected-(R6-Pad1) -> /GPA4
- R7 pad 1: unconnected-(R7-Pad1) -> /GPA5
- R8 pad 1: unconnected-(R8-Pad1) -> /GPA6
- R9 pad 1: unconnected-(R9-Pad1) -> /GPA7
- U1 pad 21: +5V -> VCC
- U2 pad 3: /LEDS_PORTB -> /pxp
- U2 pad 8: /LEDS_PORTB -> /pxp
- U3 pad 1: Net-(J3-D+) -> /GPA1
- U3 pad 2: Net-(J3-D-) -> /GPA2
- U3 pad 3: GND -> /GPA3
- U3 pad 4: unconnected-(U3-~{RTS}-Pad4) -> /GPA4
- U3 pad 5: +5V -> /GPA5
- U3 pad 6: Net-(U3-TXD) -> /GPA6
- U3 pad 7: Net-(U3-RXD) -> /GPA7
- U3 pad 8: Net-(U3-V3) -> GND
Routing:
- net /RA0/RA0: track 0.00 -> 121.6 mm, vias 0 -> 2
- net /RA3/RA5: track 0.00 -> 97.5 mm, vias 0 -> 2
- net VCC: track 0.00 -> 83.5 mm, vias 0 -> 6
- net /RA4/RA4: track 0.00 -> 80.0 mm, vias 0 -> 2
- net /RA1/RA7: track 0.00 -> 74.9 mm, vias 0 -> 1
- net /RA5/RA3: track 0.00 -> 57.6 mm
- net /RA2/RA6: track 0.00 -> 55.3 mm
- net /RC1/RB7: track 0.00 -> 52.5 mm
- net /GND/RA1: track 0.00 -> 52.5 mm, vias 0 -> 6
- net /pxp: track 0.00 -> 50.0 mm
- net /pxpcs: track 0.00 -> 49.6 mm, vias 0 -> 3
- net /RC0/VCC: track 0.00 -> 49.1 mm, vias 0 -> 6
- net /RC2/RB6: track 0.00 -> 48.2 mm
- net Net-(J1-Pin_2): track 0.00 -> 46.7 mm
- net /GPA5: track 0.00 -> 46.5 mm, vias 0 -> 1
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- added copper zone on B.Cu, net GND
- added copper zone on F.Cu, net GND
Other:
- outline, holes or cut-outs redrawn
- board text added: "ICSP"
- board text added: "ON"
- board text added: "PXP"
- board text added: "RA5"
- board text added: "RESET"
