File: PCBs/TarjetasDeDesarrollo/PectenAlpha/PectenAlphaSMD/PectenAlphaSMD.kicad_sch (KiCad schematic)
At the start: 34 parts, among them J1 ICSP, J3 USB_A, J4 PORT, J5 EXPANSION, SW1 SW_Push, SW2 SW_DIP_x04, U1 PIC_8-14-18-20, U2 D148K, U3 CH340N, U4 AMS1117-3.3, U5 74HC595, U6 74HC595

Commit message: Tarjeta Pecten
Parts:
- removed C1: C, symbol Device:C
- removed J3: USB_A, Connector_USB:USB_A_CNCTech_1001-011-01101_Horizontal, symbol Connector:USB_A
- removed J4: PORT, Connector_PinHeader_2.54mm:PinHeader_2x12_P2.54mm_Vertical, symbol Connector_Generic:Conn_02x12_Odd_Even
- removed J5: EXPANSION, Connector_PinHeader_2.54mm:PinHeader_2x08_P2.54mm_Vertical, symbol Connector_Generic:Conn_02x08_Odd_Even
- removed JP1: TX_Sel, symbol Jumper:SolderJumper_3_Open
- removed JP2: RX_Sel, symbol Jumper:SolderJumper_3_Open
- removed R16: R_US, Resistor_SMD:R_0805_2012Metric_Pad1.20x1.40mm_HandSolder, symbol Device:R_US
- removed SW2: SW_DIP_x04, Button_Switch_THT:SW_DIP_SPSTx04_Slide_6.7x11.72mm_W7.62mm_P2.54mm_LowProfile, symbol Switch:SW_DIP_x04
- removed U3: CH340N, Package_SO:JEITA_SOIC-8_3.9x4.9mm_P1.27mm, symbol Interface_USB:CH340N
- removed U6: 74HC595, symbol 74xx:74HC595
- added BZ1: Buzzer, Buzzer_Beeper:Buzzer_12x9.5RM7.6, symbol Device:Buzzer
- added J2: PectenExpansionPort, PIC_Pin_Compatible:PXP, symbol PIC_Pin_Compatible:PXP
- added Q2: PN2222A, Package_TO_SOT_THT:TO-92_Inline, symbol Transistor_BJT:PN2222A
- added R14: R_US, Resistor_SMD:R_0805_2012Metric_Pad1.20x1.40mm_HandSolder, symbol Device:R_US
- added SW3, SW4: SW_DIP_x01, Button_Switch_THT:SW_DIP_SPSTx01_Slide_6.7x4.1mm_W7.62mm_P2.54mm_LowProfile, symbol Switch:SW_DIP_x01
- added U3: 74HC595, Package_SO:SOP-16_4.4x10.4mm_P1.27mm, symbol 74xx:74HC595
- C2, C3: footprint (none) -> Capacitor_SMD:CP_Elec_5x3
- U5: footprint (none) -> Package_SO:SOP-16_4.4x10.4mm_P1.27mm
Connections:
- net LEDS_PORTB is gone; now on net pxp: U2.3 (CC), U2.8 (CC)
- net +5V: now also R15.2, BZ1.1 (+); no longer J1.5 (Pin_5), U1.21 (VDD), U5.16 (VCC)
- net GND: now also J2.2 (GND), J2.23 (GND), SW4.1, U3.8 (GND)
- net GND/RA1: now also J2.22 (NC)
- net RA0/RA0: now also J2.20 (P8), SW3.1; no longer R10.1
- net RA1/RA7: now also J2.19 (P9); no longer R11.1
- net RA2/RA6: now also J2.18 (P10); no longer R12.1
- net RA3/RA5: now also J2.7 (P2)
- net RA4/RA4: now also J1.6 (Pin_6), U1.4 (VPP), J2.6 (P1)
- net RA5/RA3: now also J2.5 (P0)
- net RB4/RB5: now also J2.15 (P13)
- net RB5/RB4: now also J2.14 (P14)
- net RB6: now also J2.13 (P15)
- net RB7: now also J2.12 (P7)
- net RC0/VCC: now also J2.4 (NC)
- net RC1/RB7: now also J2.17 (P11)
- net RC2/RB6: now also J2.16 (P12)
- net RC3/RB1: now also J2.9 (P4)
- net RC4/RB0: now also J2.8 (P3)
- net RC5/GND: now also J2.21 (NC)
- net RC6/RB2: now also J2.10 (P5)
- net RC7/RB3: now also J2.11 (P6)
- net VCC: now also J1.5 (Pin_5), U1.21 (VDD), U5.10 (~{SRCLR}), U5.16 (VCC), J2.1 (5V), J2.24 (5V), U3.10 (~{SRCLR}), U3.16 (VCC)
- net VCC/RA2: now also J2.3 (NC)
- net GPA3: now reaches R5.1
- net GPA3: now also J2.28 (XP3), U3.3 (QD)
- net pxpcs: now reaches R15.1
- net pxpcs: now also U5.13 (~{OE}), SW3.2, U3.13 (~{OE})
- net GPA4: now reaches R6.1
- net GPA4: now also J2.29 (XP4), U3.4 (QE)
- net GPA2: now reaches R4.1
- net GPA2: now also J2.27 (XP2), U3.2 (QC)
- net GPA5: now reaches R7.1
- net GPA5: now also J2.30 (XP5), U3.5 (QF)
- net GPA1: now reaches R3.1
- net GPA1: now also J2.26 (XP1), U3.1 (QB)
- net GPA0: now reaches R2.1
- net GPA0: now also J2.25 (XP0), U3.15 (QA)
- net at U5.11 (SRCLK): now also U3.11 (SRCLK)
- net at U5.14 (SER): now also U3.9 (QH')
- net GPA6: now reaches R8.1
- net GPA6: now also J2.31 (XP6), U3.6 (QG)
- net GPA7: now reaches R9.1
- net GPA7: now also J2.32 (XP7), U3.7 (QH)
- net LED RGB renamed pxp
- net pxp: now also Q2.1 (E), SW4.2
- net QA0 renamed GPB0
- net GPB0: now also R12.1, J2.40 (XP8)
- net QA1 renamed GPB1
- net GPB1: now also R11.1, J2.39 (XP9)
- net QA2 renamed GPB2
- net GPB2: now also R10.1, J2.38 (XP10)
- net QA3 renamed GPB3
- net GPB3: now also J2.37 (XP11), R14.2
- net QA4 renamed GPB4
- net GPB4: now also J2.36 (XP12)
- net QA5 renamed GPB5
- net GPB5: now also J2.35 (XP13)
- net QA6 renamed GPB6
- net GPB6: now also J2.34 (XP14)
- net QA7 renamed GPB7
- net GPB7: now also J2.33 (XP15)
- new net: Q2.2 (B), R14.1
- new net: BZ1.2 (-), Q2.3 (C)
Other:
- moved on the sheet: C2, C3, D1, D10, R1, R10, R11, R12, R13, R2, R3, R4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
